Commit message: Gazebo simulation working, simple track created

File: rviz_and_sim/urdf/car.gazebo.xacro (robot description, xacro)
@@ -11,5 +11,5 @@
           <sensor name='gpu_lidar' type='gpu_lidar'>
             <topic>scan</topic>
-            <update_rate>10</update_rate>
+            <update_rate>30</update_rate>
             <lidar>
                 <scan>
@@ -40,13 +40,20 @@
     <gazebo>
       <plugin
-        filename="libignition-gazebo-diff-drive-system.so"
-        name="ignition::gazebo::systems::DiffDrive">
+        filename="libignition-gazebo6-ackermann-steering-system.so"
+        name="ignition::gazebo::systems::AckermannSteering">
         <left_joint>rear_left_wheel_joint</left_joint>
         <right_joint>rear_right_wheel_joint</right_joint>
-        <wheel_separation>0.34</wheel_separation>
+        <left_steering_joint>rear_left_wheel_joint</left_steering_joint>
+        <right_steering_joint>rear_right_wheel_joint</right_steering_joint>
+        <wheel_separation>0.28</wheel_separation>
+        <kingpin_width>0.28</kingpin_width>
+        <wheel_base>0.28</wheel_base>
+        <steering_limit>0.5</steering_limit>
         <wheel_radius>0.054</wheel_radius>
         <odom_publish_frequency>30</odom_publish_frequency>
-        <frame_id>odom</frame_id>
-        <child_frame_id>base_link</child_frame_id>
+        <min_velocity>0</min_velocity>
+        <max_velocity>40</max_velocity>
+        <min_acceleration>0</min_acceleration>
+        <max_acceleration>5</max_acceleration>
       </plugin>
       <plugin

File: rviz_and_sim/urdf/car.urdf.xacro (robot description, xacro)
@@ -161,12 +161,12 @@
       <link name="front_left_hub">
         <inertial>
-          <mass value="0.0" />
-          <inertia
-            ixx="0"
-            ixy="0"
-            ixz="0"
-            iyy="0"
-            iyz="0"
-            izz="0"
+          <mass value="0.0001" />
+          <inertia
+            ixx="0.001"
+            ixy="0"
+            ixz="0"
+            iyy="0.001"
+            iyz="0"
+            izz="0.001"
           />
         </inertial>
@@ -179,12 +179,12 @@
       <link name="front_right_hub">
         <inertial>
-          <mass value="0.0" />
-          <inertia
-            ixx="0"
-            ixy="0"
-            ixz="0"
-            iyy="0"
-            iyz="0"
-            izz="0"
+          <mass value="0.0001" />
+          <inertia
+            ixx="0.001"
+            ixy="0"
+            ixz="0"
+            iyy="0.001"
+            iyz="0"
+            izz="0.001"
           />
         </inertial>
@@ -211,4 +211,9 @@
         <child link="rear_right_wheel" />
         <axis xyz="0 0 1" />
+      </joint>
+      <joint name="fixed_rear_axle" type="fixed">
+        <origin xyz="0.0 -0 0.0" rpy="0 0 0" />
+        <parent link="rear_left_wheel" />
+        <child link="rear_right_wheel" />
       </joint>
       <joint name="front_left_wheel_joint" type="continuous">

Commit message: created track mapping package to map track

File: rviz_and_sim/urdf/car.gazebo.xacro (robot description, xacro)
@@ -44,14 +44,16 @@
         <left_joint>rear_left_wheel_joint</left_joint>
         <right_joint>rear_right_wheel_joint</right_joint>
-        <left_steering_joint>rear_left_wheel_joint</left_steering_joint>
-        <right_steering_joint>rear_right_wheel_joint</right_steering_joint>
+        <left_steering_joint>front_left_hub_joint</left_steering_joint>
+        <right_steering_joint>front_right_hub_joint</right_steering_joint>
         <wheel_separation>0.28</wheel_separation>
         <kingpin_width>0.28</kingpin_width>
         <wheel_base>0.28</wheel_base>
-        <steering_limit>0.5</steering_limit>
+        <steering_limit>0.25</steering_limit>
         <wheel_radius>0.054</wheel_radius>
         <odom_publish_frequency>30</odom_publish_frequency>
+        <frame_id>odom</frame_id>
+        <child_frame_id>base_link</child_frame_id>
         <min_velocity>0</min_velocity>
-        <max_velocity>40</max_velocity>
+        <max_velocity>10</max_velocity>
         <min_acceleration>0</min_acceleration>
         <max_acceleration>5</max_acceleration>

File: rviz_and_sim/urdf/car.urdf.xacro (robot description, xacro)
@@ -14,7 +14,7 @@
         </inertial>
         <visual>
-          <origin xyz="-0 0 0.08" rpy="0 -0 0"/>
-          <geometry>
-            <box size="0.35 0.08 0.06" />
+          <origin xyz="-0 0 0.09" rpy="0 -0 0"/>
+          <geometry>
+            <box size="0.34 0.1 0.1" />
           </geometry>
           <material name="pla">
@@ -25,5 +25,5 @@
           <origin xyz="-0 0 0.08" rpy="0 -0 0"/>
           <geometry>
-            <box size="0.35 0.08 0.06" />
+            <box size="0.35 0.1 0.1" />
           </geometry>
         </collision>
@@ -56,5 +56,7 @@
             <cylinder radius="0.05" length="0.04" />
           </geometry>
-          <material name="pla" />
+          <material name="pla_black">
+             <color rgba="0.3 0.3 0.3 1.0" />
+          </material>
         </visual>
       </link>
@@ -196,5 +198,5 @@
       </link>
       <joint name="lidar_sensor_joint" type="fixed">
-        <origin xyz="0.1 -0 0.12" rpy="0 0 0" />
+        <origin xyz="0.05 -0 0.16" rpy="0 0 0" />
         <parent link="base_link" />
         <child link="base_laser" />
@@ -211,9 +213,4 @@
         <child link="rear_right_wheel" />
         <axis xyz="0 0 1" />
-      </joint>
-      <joint name="fixed_rear_axle" type="fixed">
-        <origin xyz="0.0 -0 0.0" rpy="0 0 0" />
-        <parent link="rear_left_wheel" />
-        <child link="rear_right_wheel" />
       </joint>
       <joint name="front_left_wheel_joint" type="continuous">
