Commit message: Added suspension to URDF and simulation

File: rviz_description/urdf/car_old.urdf (robot description, URDF)
Before this commit: robot car, 14 links, 13 joints
Links:
- removed link front_left_suspension
- removed link front_right_suspension
- removed link rear_left_suspension
- removed link rear_right_suspension
- link front_left_hub: geometry collision box size=0.05 0.08 0.05
- link front_right_hub: geometry collision box size=0.05 0.08 0.05
Joints:
- removed joint front_left_suspension_joint
- removed joint front_right_suspension_joint
- removed joint rear_left_suspension_joint
- removed joint rear_right_suspension_joint
- joint front_left_hub_joint: limit lower=-0.5 upper=0.5 effort=1000. velocity=2.0 -> lower=-0.5 upper=0.5 effort=1000 velocity=100.0; parent front_left_suspension -> base_link
- joint front_right_hub_joint: limit lower=-0.5 upper=0.5 effort=1000. velocity=2.0 -> lower=-0.5 upper=0.5 effort=1000 velocity=100.0; parent front_right_suspension -> base_link
- joint rear_left_wheel_joint: parent rear_left_suspension -> base_link
- joint rear_right_wheel_joint: parent rear_right_suspension -> base_link

File: rviz_description/urdf/car_old.urdf.xacro (robot description, xacro)
@@ -1,5 +1,5 @@
 <robot name="car" xmlns:xacro="http://www.ros.org/wiki/xacro">
       <material name="pla">
-          <color rgba="0.4 0.1 0.6 1.0" />
+          <color rgba="0.5 0.1 0.5 1.0" />
       </material>
       <material name="pla_black">
@@ -14,5 +14,5 @@
       <link name="base_link">
         <inertial>
-          <origin xyz="0 -0 0.1" rpy="0 -0 0"/>
+          <origin xyz="0 -0 0.01" rpy="0 -0 0"/>
           <mass value="1.2" />
           <inertia
@@ -26,5 +26,5 @@
         </inertial>
         <visual>
-          <origin xyz="-0 0 0.1" rpy="0 -0 0"/>
+          <origin xyz="-0 0 0.095" rpy="0 -0 0"/>
           <geometry>
             <box size="0.3 0.08 0.1" />
@@ -203,5 +203,5 @@
         <collision name='collision'>
           <geometry>
-            <box size="0.001 0.001 0.001" />
+            <box size="0.05 0.08 0.05" />
           </geometry>
         </collision>
@@ -221,59 +221,7 @@
         <collision name='collision'>
           <geometry>
-            <box size="0.001 0.001 0.001" />
-          </geometry>
-        </collision>
-      </link>
-      <link name="front_right_suspension">
-        <inertial>
-          <mass value="0.0" />
-          <inertia
-            ixx="0.0"
-            ixy="0"
-            ixz="0"
-            iyy="0.0"
-            iyz="0"
-            izz="0.0"
-          />
-        </inertial>
-      </link>
-      <link name="front_left_suspension">
-        <inertial>
-          <mass value="0.0" />
-          <inertia
-            ixx="0.0"
-            ixy="0"
-            ixz="0"
-            iyy="0.0"
-            iyz="0"
-            izz="0.0"
-          />
-        </inertial>
-      </link>
-      <link name="rear_right_suspension">
-        <inertial>
-          <mass value="0.0" />
-          <inertia
-            ixx="0.0"
-            ixy="0"
-            ixz="0"
-            iyy="0.0"
-            iyz="0"
-            izz="0.0"
-          />
-        </inertial>
-      </link>
-      <link name="rear_left_suspension">
-        <inertial>
-          <mass value="0.0" />
-          <inertia
-            ixx="0.0"
-            ixy="0"
-            ixz="0"
-            iyy="0.0"
-            iyz="0"
-            izz="0.0"
-          />
-        </inertial>
+            <box size="0.05 0.08 0.05" />
+          </geometry>
+        </collision>
       </link>
       <joint name="lidar_sensor_joint" type="fixed">
@@ -289,5 +237,5 @@
       <joint name="rear_left_wheel_joint" type="continuous">
         <origin xyz="-0.14 0.13 0.054" rpy="-1.5707 0 0" />
-        <parent link="rear_left_suspension" />
+        <parent link="base_link" />
         <child link="rear_left_wheel" />
         <axis xyz="0 0 1" />
@@ -295,5 +243,5 @@
       <joint name="rear_right_wheel_joint" type="continuous">
         <origin xyz="-0.14 -0.13 0.054" rpy="-1.5707 0 0" />
-        <parent link="rear_right_suspension" />
+        <parent link="base_link" />
         <child link="rear_right_wheel" />
         <axis xyz="0 0 1" />
@@ -313,6 +261,6 @@
       <joint name="front_left_hub_joint" type="revolute">
         <origin xyz="0.14 0.11 0.054" rpy="0 0 0" />
-        <limit effort="1000." upper="0.5" lower="-0.5" velocity="5.0" />
-        <parent link="front_left_suspension" />
+        <limit upper="0.5" lower="-0.5" velocity="2.0" />
+        <parent link="base_link" />
         <child link="front_left_hub" />
         <axis xyz="0 0 1" />
@@ -320,36 +268,8 @@
       <joint name="front_right_hub_joint" type="revolute">
         <origin xyz="0.14 -0.11 0.054" rpy="0 0 0" />
-        <limit effort="1000." upper="0.5" lower="-0.5" velocity="5.0" />
-        <parent link="front_right_suspension" />
+        <limit upper="0.5" lower="-0.5" velocity="2.0" />
+        <parent link="base_link" />
         <child link="front_right_hub" />
         <axis xyz="0 0 1" />
       </joint>
-      <joint name="front_right_suspension_joint" type="prismatic">
-        <origin xyz="0.0 -0.0 0.0" rpy="0 0 0" />
-        <limit effort="1000." upper="0.04" lower="0." velocity="100."/>
-        <parent link="base_link" />
-        <child link="front_right_suspension" />
-        <axis xyz="0 0 1" />
-      </joint>
-      <joint name="front_left_suspension_joint" type="prismatic">
-        <origin xyz="0.0 -0.0 0.0" rpy="0 0 0" />
-        <limit effort="1000." upper="0.04" lower="0." velocity="100."/>
-        <parent link="base_link" />
-        <child link="front_left_suspension" />
-        <axis xyz="0 0 1" />
-      </joint>
-      <joint name="rear_right_suspension_joint" type="prismatic">
-        <origin xyz="0.0 -0.0 0.0" rpy="0 0 0" />
-        <limit effort="1000." upper="0.04" lower="0." velocity="100."/>
-        <parent link="base_link" />
-        <child link="rear_right_suspension" />
-        <axis xyz="0 0 1" />
-      </joint>
-      <joint name="rear_left_suspension_joint" type="prismatic">
-        <origin xyz="0.0 -0.0 0.0" rpy="0 0 0" />
-        <limit effort="1000." upper="0.04" lower="0." velocity="100."/>
-        <parent link="base_link" />
-        <child link="rear_left_suspension" />
-        <axis xyz="0 0 1" />
-      </joint>
 </robot>
