Commit message: added updated URDF to simulation

File: rviz_description/urdf/car.urdf (robot description, URDF)
Before this commit: robot car, 14 links, 13 joints
Links:
- added link chassis_visual; collision mesh filename=package://rviz_description/meshes/40mm_standoff.stl; collision mesh filename=package://rviz_description/meshes/40mm_standoff.stl
- link base_laser: geometry collision cylinder length=0.025 radius=0.035; visual cylinder length=0.025 radius=0.035
- link base_link: geometry 
- link camera_link: geometry collision mesh filename=package://rviz_description/meshes/d435.stl scale=0.001 0.001 0.001; visual mesh filename=package://rviz_description/meshes/d435.stl scale=0.001 0.001 0.001
- link front_left_wheel: geometry collision cylinder length=0.043 radius=0.054; visual mesh filename=package://rviz_description/meshes/wheel_110mm.stl
- link front_right_wheel: geometry collision cylinder length=0.043 radius=0.054; visual mesh filename=package://rviz_description/meshes/wheel_110mm.stl
- link rear_left_wheel: geometry collision cylinder length=0.043 radius=0.054; visual mesh filename=package://rviz_description/meshes/wheel_110mm.stl
- link rear_right_wheel: geometry collision cylinder length=0.043 radius=0.054; visual mesh filename=package://rviz_description/meshes/wheel_110mm.stl
Joints:
- added joint base_chassis_visual: type fixed, parent base_link, child chassis_visual, origin xyz=-0.055 -0.0081385453814205033218 0.08 rpy=0.0 0.0 0.0
- joint camera_sensor_joint: origin xyz=0.14 -0 0.13 rpy=0 0 0 -> xyz=0.1575 -0 0.145 rpy=1.5707 0 1.5707
- joint front_left_hub_joint: limit lower=-0.5 upper=0.5 effort=1000. velocity=2.0 -> lower=-0.5 upper=0.5 effort=1000. velocity=5.0; origin xyz=0.14 0.11 0.054 rpy=0 0 0 -> xyz=0.138 0.125 0.054 rpy=0 0 0
- joint front_left_wheel_joint: origin xyz=-0 0.02 0 rpy=-1.5707 0 0 -> xyz=-0 0.0415 0 rpy=-1.5707 0 3.1415926
- joint front_right_hub_joint: limit lower=-0.5 upper=0.5 effort=1000. velocity=2.0 -> lower=-0.5 upper=0.5 effort=1000. velocity=5.0; origin xyz=0.14 -0.11 0.054 rpy=0 0 0 -> xyz=0.138 -0.125 0.054 rpy=0 0 0
- joint front_right_wheel_joint: origin xyz=-0 -0.02 0 rpy=-1.5707 0 0 -> xyz=-0 -0.0415 0 rpy=-1.5707 0 0
- joint lidar_sensor_joint: origin xyz=0.08 -0 0.18 rpy=0 0 0 -> xyz=0.08 -0 0.215 rpy=0 0 0
- joint rear_left_wheel_joint: origin xyz=-0.14 0.13 0.054 rpy=-1.5707 0 0 -> xyz=-0.145 0.1665 0.054 rpy=-1.5707 0 3.1415926
- joint rear_right_wheel_joint: origin xyz=-0.14 -0.13 0.054 rpy=-1.5707 0 0 -> xyz=-0.145 -0.1665 0.054 rpy=-1.5707 0 0

File: rviz_description/urdf/car.urdf.xacro (robot description, xacro)
@@ -4,5 +4,5 @@
       </material>
       <material name="pla_black">
-          <color rgba="0.2 0.2 0.2 1.0" />
+          <color rgba="0.05 0.05 0.05 1.0" />
       </material>
       <material name="aluminum">
@@ -28,4 +28,18 @@
       <link name="chassis_visual">
         <collision>
+        <origin xyz="0.19593310870444985428 -0.023861467502207221042 0.032178813240731983514" rpy="-3.2732333544360483958e-15 0.2617993877991453 -3.141592653589758477" />
+        <geometry>
+        <mesh filename="package://rviz_description/meshes/a01.stl"/>
+        </geometry>
+        </collision>
+        <visual>
+        <origin xyz="0.19593310870444985428 -0.023861467502207221042 0.032178813240731983514" rpy="-3.2732333544360483958e-15 0.2617993877991453 -3.141592653589758477" />
+        <geometry>
+        <mesh filename="package://rviz_description/meshes/a01.stl"/>
+        </geometry>
+        <material name="pla">
+        </material>
+        </visual>
+        <collision>
         <origin xyz="0.041230177353335013823 0.0081385453814205033218 0.046435964631839833638" rpy="-3.3417470151423496181e-15 1.5267451514876481878e-15 -1.5707963267948608088" />
         <geometry>
@@ -34,5 +48,5 @@
         </collision>
         <visual>
-        <material name="pla">
+        <material name="pla_black">
         </material>
         <origin xyz="0.041230177353335013823 0.0081385453814205033218 0.046435964631839833638" rpy="-3.3417470151423496181e-15 1.5267451514876481878e-15 -1.5707963267948608088" />
@@ -42,16 +56,4 @@
         </visual>
         <collision>
-        <origin xyz="0.19593310870444985428 -0.023861467502207221042 0.032178813240731983514" rpy="-3.2732333544360483958e-15 0.2617993877991453 -3.141592653589758477" />
-        <geometry>
-        <mesh filename="package://rviz_description/meshes/a01.stl"/>
-        </geometry>
-        </collision>
-        <visual>
-        <origin xyz="0.19593310870444985428 -0.023861467502207221042 0.032178813240731983514" rpy="-3.2732333544360483958e-15 0.2617993877991453 -3.141592653589758477" />
-        <geometry>
-        <mesh filename="package://rviz_description/meshes/a01.stl"/>
-        </geometry>
-        </visual>
-        <collision>
         <origin xyz="0.04123017735333503464 0.0081385453814205102607 0.046435964631839812822" rpy="-3.3417470151423496181e-15 1.5267451514876481878e-15 -1.5707963267948608088" />
         <geometry>
@@ -64,4 +66,6 @@
         <mesh filename="package://rviz_description/meshes/lidar_hat.stl" />
         </geometry>
+        <material name="pla_black">
+        </material>
         </visual>
         <collision>
@@ -76,4 +80,6 @@
         <mesh filename="package://rviz_description/meshes/a07.stl"/>
         </geometry>
+        <material name="pla">
+        </material>
         </visual>
         <collision>
@@ -88,4 +94,6 @@
         <mesh filename="package://rviz_description/meshes/cover_plate.stl"/>
         </geometry>
+        <material name="pla_black">
+        </material>
         </visual>
         <collision>
@@ -100,4 +108,6 @@
         <mesh filename="package://rviz_description/meshes/b01.stl"/>
         </geometry>
+        <material name="pla">
+        </material>
         </visual>
         <collision>
@@ -112,4 +122,6 @@
         <mesh filename="package://rviz_description/meshes/a09.stl"/>
         </geometry>
+        <material name="pla">
+        </material>
         </visual>
         <collision>
@@ -119,4 +131,6 @@
         </geometry>
         </collision>
+        <material name="pla_black">
+        </material>
         <visual>
         <origin xyz="0.10673017735333342748 0.052638545381422860436 0.046435964631839680983" rpy="1.526745151487648385e-15 3.3417470151423492237e-15 3.5884533940292959508e-14" />
@@ -136,4 +150,6 @@
         <mesh filename="package://rviz_description/meshes/b12-t.stl"/>
         </geometry>
+        <material name="pla_black">
+        </material>
         </visual>
         <collision>
@@ -148,4 +164,6 @@
         <mesh filename="package://rviz_description/meshes/40mm_standoff.stl"/>
         </geometry>
+        <material name="pla_black">
+        </material>
         </visual>
         <collision>
@@ -160,4 +178,6 @@
         <mesh filename="package://rviz_description/meshes/b08-t.stl"/>
         </geometry>
+        <material name="pla">
+        </material>
         </visual>
         <collision>
@@ -172,4 +192,6 @@
         <mesh filename="package://rviz_description/meshes/b07-t.stl"/>
         </geometry>
+        <material name="pla">
+        </material>
         </visual>
         <collision>
@@ -184,4 +206,6 @@
         <mesh filename="package://rviz_description/meshes/40mm_standoff.stl"/>
         </geometry>
+        <material name="pla_black">
+        </material>
         </visual>
         <collision>
@@ -196,4 +220,6 @@
         <mesh filename="package://rviz_description/meshes/40mm_standoff.stl"/>
         </geometry>
+        <material name="pla_black">
+        </material>
         </visual>
         <collision>
@@ -208,4 +234,6 @@
         <mesh filename="package://rviz_description/meshes/part_2.stl"/>
         </geometry>
+        <material name="pla">
+        </material>
         </visual>
         <collision>
@@ -220,4 +248,6 @@
         <mesh filename="package://rviz_description/meshes/b13-t.stl"/>
         </geometry>
+        <material name="pla">
+        </material>
         </visual>
         <collision>
@@ -232,4 +262,6 @@
         <mesh filename="package://rviz_description/meshes/a08.stl"/>
         </geometry>
+        <material name="pla">
+        </material>
         </visual>
         <collision>
@@ -244,4 +276,6 @@
         <mesh filename="package://rviz_description/meshes/40mm_standoff.stl"/>
         </geometry>
+        <material name="pla_black">
+        </material>
         </visual>
         <collision>
@@ -256,4 +290,6 @@
         <mesh filename="package://rviz_description/meshes/b06.stl"/>
         </geometry>
+        <material name="pla">
+        </material>
         </visual>
         <collision>
@@ -268,4 +304,6 @@
         <mesh filename="package://rviz_description/meshes/jetson_retainer.stl"/>
         </geometry>
+        <material name="pla_black">
+        </material>
         </visual>
         <collision>
@@ -280,4 +318,6 @@
         <mesh filename="package://rviz_description/meshes/40mm_standoff.stl"/>
         </geometry>
+        <material name="pla_black">
+        </material>
         </visual>
         <collision>
@@ -292,4 +332,6 @@
         <mesh filename="package://rviz_description/meshes/b10-t.stl"/>
         </geometry>
+        <material name="pla">
+        </material>
         </visual>
         <collision>
@@ -304,4 +346,6 @@
         <mesh filename="package://rviz_description/meshes/40mm_standoff.stl"/>
         </geometry>
+        <material name="pla_black">
+        </material>
         </visual>
         <collision>
@@ -316,4 +360,6 @@
         <mesh filename="package://rviz_description/meshes/realsense_mount.stl"/>
         </geometry>
+        <material name="pla_black">
+        </material>
         </visual>
         <collision>
@@ -328,4 +374,6 @@
         <mesh filename="package://rviz_description/meshes/camera_mount.stl"/>
         </geometry>
+        <material name="pla_black">
+        </material>
         </visual>
         <collision>
@@ -340,4 +388,6 @@
         <mesh filename="package://rviz_description/meshes/40mm_standoff.stl"/>
         </geometry>
+        <material name="pla_black">
+        </material>
         </visual>
         <collision>
@@ -352,4 +402,6 @@
         <mesh filename="package://rviz_description/meshes/40mm_standoff.stl"/>
         </geometry>
+        <material name="pla_black">
+        </material>
         </visual>
         <collision>
@@ -364,4 +416,6 @@
         <mesh filename="package://rviz_description/meshes/b03.stl"/>
         </geometry>
+        <material name="pla">
+        </material>
         </visual>
         <collision>
@@ -391,4 +445,6 @@
         <mesh filename="package://rviz_description/meshes/a01.stl"/>
         </geometry>
+        <material name="pla">
+        </material>
         </visual>
         <collision>
@@ -403,4 +459,6 @@
         <mesh filename="package://rviz_description/meshes/40mm_standoff.stl"/>
         </geometry>
+        <material name="pla_black">
+        </material>
         </visual>
         <collision>
@@ -415,4 +473,6 @@
         <mesh filename="package://rviz_description/meshes/standoff.stl"/>
         </geometry>
+        <material name="pla_black">
+        </material>
         </visual>
         <collision>
@@ -427,4 +487,6 @@
         <mesh filename="package://rviz_description/meshes/b04.stl"/>
         </geometry>
+        <material name="pla">
+        </material>
         </visual>
         <collision>
@@ -439,4 +501,6 @@
         <mesh filename="package://rviz_description/meshes/b11-t.stl"/>
         </geometry>
+        <material name="pla">
+        </material>
         </visual>
         <collision>
@@ -451,4 +515,6 @@
         <mesh filename="package://rviz_description/meshes/standoff-_copy.stl"/>
         </geometry>
+        <material name="pla_black">
+        </material>
         </visual>
         <collision>
@@ -463,4 +529,6 @@
         <mesh filename="package://rviz_description/meshes/b02.stl"/>
         </geometry>
+        <material name="pla">
+        </material>
         </visual>
         <collision>
@@ -475,4 +543,6 @@
         <mesh filename="package://rviz_description/meshes/b09.stl"/>
         </geometry>
+        <material name="pla">
+        </material>
         </visual>
         <collision>
@@ -487,4 +557,6 @@
         <mesh filename="package://rviz_description/meshes/b05.stl"/>
         </geometry>
+        <material name="pla">
+        </material>
         </visual>
       </link>
@@ -557,10 +629,36 @@
         </visual>
         <collision name='collision'>
+          <origin xyz="0 0 0.0215" rpy="0 0 0" />
+          <geometry>
+            <cylinder radius="0.054" length="0.043" />
+          </geometry>
+        </collision>
+      </link>
+      <link name="rear_right_wheel">
+        <inertial>
+          <mass value="0.1" />
+          <inertia
+            ixx="0.0000729"
+            ixy="0"
+            ixz="0"
+            iyy="0.0000729"
+            iyz="0"
+            izz="0.0001458"
+          />
+        </inertial>
+        <visual>
           <geometry>
             <mesh filename="package://rviz_description/meshes/wheel_110mm.stl"/>
           </geometry>
-        </collision>
-      </link>
-      <link name="rear_right_wheel">
+          <material name="rubber"/>
+        </visual>
+        <collision name='collision'>
+          <origin xyz="0 0 0.0215" rpy="0 0 0" />
+          <geometry>
+            <cylinder radius="0.054" length="0.043" />
+          </geometry>
+        </collision>
+      </link>
+      <link name="front_left_wheel">
         <inertial>
           <mass value="0.1" />
@@ -581,54 +679,32 @@
         </visual>
         <collision name='collision'>
+          <origin xyz="0 0 0.0215" rpy="0 0 0" />
+          <geometry>
+            <cylinder radius="0.054" length="0.043" />
+          </geometry>
+        </collision>
+      </link>
+      <link name="front_right_wheel">
+        <inertial>
+          <mass value="0.1" />
+          <inertia
+            ixx="0.0000729"
+            ixy="0"
+            ixz="0"
+            iyy="0.0000729"
+            iyz="0"
+            izz="0.0001458"
+          />
+        </inertial>
+        <visual>
           <geometry>
             <mesh filename="package://rviz_description/meshes/wheel_110mm.stl"/>
           </geometry>
-        </collision>
-      </link>
-      <link name="front_left_wheel">
-        <inertial>
-          <mass value="0.1" />
-          <inertia
-            ixx="0.0000729"
-            ixy="0"
-            ixz="0"
-            iyy="0.0000729"
-            iyz="0"
-            izz="0.0001458"
-          />
-        </inertial>
-        <visual>
-          <geometry>
-            <mesh filename="package://rviz_description/meshes/wheel_110mm.stl"/>
-          </geometry>
-          <material name="rubber"/>
+          <material name="rubber" />
         </visual>
         <collision name='collision'>
-          <geometry>
-            <mesh filename="package://rviz_description/meshes/wheel_110mm.stl"/>
-          </geometry>
-        </collision>
-      </link>
-      <link name="front_right_wheel">
-        <inertial>
-          <mass value="0.1" />
-          <inertia
-            ixx="0.0000729"
-            ixy="0"
-            ixz="0"
-            iyy="0.0000729"
-            iyz="0"
-            izz="0.0001458"
-          />
-        </inertial>
-        <visual>
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
Commit message: Added lidar to sim, robot can now map with SlamToolbox

File: rviz_description/urdf/car.urdf (robot description, URDF)
Before this commit: robot car, 15 links, 14 joints
Joints:
- joint base_chassis_visual: origin xyz=-0.055 -0.0081385453814205033218 0.08 rpy=0.0 0.0 0.0 -> xyz=-0.055 -0.0081385453814205033218 0.09 rpy=0.0 0.0 0.0
- joint front_left_suspension_joint: limit lower=0. upper=0.04 effort=1000. velocity=100. -> lower=0. upper=0.04 effort=1000. velocity=400.
- joint front_right_suspension_joint: limit lower=0. upper=0.04 effort=1000. velocity=100. -> lower=0. upper=0.04 effort=1000. velocity=400.
- joint rear_left_suspension_joint: limit lower=0. upper=0.04 effort=1000. velocity=100. -> lower=0. upper=0.04 effort=1000. velocity=400.
- joint rear_right_suspension_joint: limit lower=0. upper=0.04 effort=1000. velocity=100. -> lower=0. upper=0.04 effort=1000. velocity=400.

File: rviz_description/urdf/car.urdf.xacro (robot description, xacro)
@@ -14,5 +14,5 @@
       <link name="base_link">
         <inertial>
-          <origin xyz="0 -0 0.1" rpy="0 -0 0"/>
+          <origin xyz="0 -0 0.11" rpy="0 -0 0"/>
           <mass value="1.2" />
           <inertia
@@ -806,5 +806,5 @@
         <parent link="base_link"/>
         <child link="chassis_visual"/>
-        <origin xyz="-0.055 -0.0081385453814205033218 0.08" rpy="0.0 0.0 0.0" />
+        <origin xyz="-0.055 -0.0081385453814205033218 0.09" rpy="0.0 0.0 0.0" />
      </joint>
       <joint name="lidar_sensor_joint" type="fixed">
@@ -858,5 +858,5 @@
       <joint name="front_right_suspension_joint" type="prismatic">
         <origin xyz="0.0 -0.0 0.0" rpy="0 0 0" />
-        <limit effort="1000." upper="0.04" lower="0." velocity="100."/>
+        <limit effort="1000." upper="0.04" lower="0." velocity="400."/>
         <parent link="base_link" />
         <child link="front_right_suspension" />
@@ -865,5 +865,5 @@
       <joint name="front_left_suspension_joint" type="prismatic">
         <origin xyz="0.0 -0.0 0.0" rpy="0 0 0" />
-        <limit effort="1000." upper="0.04" lower="0." velocity="100."/>
+        <limit effort="1000." upper="0.04" lower="0." velocity="400."/>
         <parent link="base_link" />
         <child link="front_left_suspension" />
@@ -872,5 +872,5 @@
       <joint name="rear_right_suspension_joint" type="prismatic">
         <origin xyz="0.0 -0.0 0.0" rpy="0 0 0" />
-        <limit effort="1000." upper="0.04" lower="0." velocity="100."/>
+        <limit effort="1000." upper="0.04" lower="0." velocity="400."/>
         <parent link="base_link" />
         <child link="rear_right_suspension" />
@@ -879,5 +879,5 @@
       <joint name="rear_left_suspension_joint" type="prismatic">
         <origin xyz="0.0 -0.0 0.0" rpy="0 0 0" />
-        <limit effort="1000." upper="0.04" lower="0." velocity="100."/>
+        <limit effort="1000." upper="0.04" lower="0." velocity="400."/>
         <parent link="base_link" />
         <child link="rear_left_suspension" />
