Commit message: added camera link to urdf, created mode_node, added mode control to controller and control_servos

File: rviz_description/urdf/car.urdf.xacro (robot description, xacro)
@@ -2,5 +2,5 @@
       <link name="base_link">
         <inertial>
-          <origin xyz="0 -0 0.08" rpy="0 -0 0"/>
+          <origin xyz="0 -0 0.01" rpy="0 -0 0"/>
           <mass value="1.14395" />
           <inertia
@@ -14,7 +14,7 @@
         </inertial>
         <visual>
-          <origin xyz="-0 0 0.09" rpy="0 -0 0"/>
-          <geometry>
-            <box size="0.34 0.1 0.1" />
+          <origin xyz="-0 0 0.095" rpy="0 -0 0"/>
+          <geometry>
+            <box size="0.3 0.08 0.1" />
           </geometry>
           <material name="pla">
@@ -23,7 +23,7 @@
         </visual>
         <collision>
-          <origin xyz="-0 0 0.08" rpy="0 -0 0"/>
-          <geometry>
-            <box size="0.35 0.1 0.1" />
+          <origin xyz="-0 0 0.1" rpy="0 -0 0"/>
+          <geometry>
+            <box size="0.34 0.1 0.1" />
           </geometry>
         </collision>
@@ -33,5 +33,5 @@
              <parent link="base_link"/>
              <child link="base_footprint"/>
-             <origin xyz="0.0 0.0 -0.15" rpy="0.0 0.0 0.0" />
+             <origin xyz="0.0 0.0 -0.0" rpy="0.0 0.0 0.0" />
      </joint>
       <link name="base_laser">
@@ -61,4 +61,30 @@
         </visual>
       </link>
+      <link name="camera_link">
+        <inertial>
+          <mass value="0.072"/>
+          <inertia
+            ixx="0.000166667"
+            iyy="0.000166667"
+            izz="0.000166667"
+            ixy="0.0"
+            ixz="0.0"
+            iyz="0.0"
+          />
+        </inertial>
+        <collision>
+          <geometry>
+            <box size="0.025 0.09 0.025" />
+          </geometry>
+        </collision>
+        <visual>
+          <geometry>
+            <box size="0.025 0.09 0.025" />
+          </geometry>
+          <material name="aluminum">
+             <color rgba="0.75 0.75 0.75 1.0" />
+          </material>
+        </visual>
+      </link>
       <link name="rear_left_wheel">
         <inertial>
@@ -198,7 +224,12 @@
       </link>
       <joint name="lidar_sensor_joint" type="fixed">
-        <origin xyz="0.05 -0 0.16" rpy="0 0 0" />
+        <origin xyz="0.08 -0 0.18" rpy="0 0 0" />
         <parent link="base_link" />
         <child link="base_laser" />
+      </joint>
+      <joint name="camera_sensor_joint" type="fixed">
+        <origin xyz="0.14 -0 0.13" rpy="0 0 0" />
+        <parent link="base_link" />
+        <child link="camera_link" />
       </joint>
       <joint name="rear_left_wheel_joint" type="continuous">

Commit message: Modified URDF and launch files, create simulate node for imulations in isaacsim

File: rviz_description/urdf/car.urdf.xacro (robot description, xacro)
@@ -1,14 +1,26 @@
 <robot name="car" xmlns:xacro="http://www.ros.org/wiki/xacro">
+      <material name="pla">
+          <color rgba="0.5 0.1 0.5 1.0" />
+      </material>
+      <material name="pla_black">
+          <color rgba="0.3 0.3 0.3 1.0" />
+      </material>
+      <material name="aluminum">
+          <color rgba="0.75 0.75 0.75 1.0" />
+      </material>
+      <material name="rubber">
+          <color rgba="0.1 0.1 0.1 1" />
+      </material>
       <link name="base_link">
         <inertial>
           <origin xyz="0 -0 0.01" rpy="0 -0 0"/>
-          <mass value="1.14395" />
-          <inertia
-            ixx="0.126164"
-            ixy="0"
-            ixz="0"
-            iyy="0.416519"
-            iyz="0"
-            izz="0.481014"
+          <mass value="1.2" />
+          <inertia
+            ixx="0.00164"
+            ixy="0"
+            ixz="0"
+            iyy="0.01"
+            iyz="0"
+            izz="0.00964"
           />
         </inertial>
@@ -18,7 +30,5 @@
             <box size="0.3 0.08 0.1" />
           </geometry>
-          <material name="pla">
-             <color rgba="0.5 0.1 0.5 1.0" />
-          </material>
+          <material name="pla"/>
         </visual>
         <collision>
@@ -37,9 +47,9 @@
       <link name="base_laser">
         <inertial>
-          <mass value="0.1"/>
-          <inertia
-            ixx="0.000166667"
-            iyy="0.000166667"
-            izz="0.000166667"
+          <mass value="0.0"/>
+          <inertia
+            ixx="0.0"
+            iyy="0.0"
+            izz="0.0"
             ixy="0.0"
             ixz="0.0"
@@ -56,16 +66,14 @@
             <cylinder radius="0.05" length="0.04" />
           </geometry>
-          <material name="pla_black">
-             <color rgba="0.3 0.3 0.3 1.0" />
-          </material>
+          <material name="pla_black"/>
         </visual>
       </link>
       <link name="camera_link">
         <inertial>
-          <mass value="0.072"/>
-          <inertia
-            ixx="0.000166667"
-            iyy="0.000166667"
-            izz="0.000166667"
+          <mass value="0.0"/>
+          <inertia
+            ixx="0.0"
+            iyy="0.0"
+            izz="0.0"
             ixy="0.0"
             ixz="0.0"
@@ -79,31 +87,27 @@
         </collision>
         <visual>
-          <geometry>
+          <geometry>001
             <box size="0.025 0.09 0.025" />
           </geometry>
-          <material name="aluminum">
-             <color rgba="0.75 0.75 0.75 1.0" />
-          </material>
+          <material name="aluminum"/>
         </visual>
       </link>
       <link name="rear_left_wheel">
         <inertial>
-          <mass value="2.0" />
-          <inertia
-            ixx="0.145833"
-            ixy="0"
-            ixz="0"
-            iyy="0.145833"
-            iyz="0"
-            izz="0.125"
-          />
-        </inertial>
-        <visual>
-          <geometry>
-            <cylinder radius="0.054" length="0.043" />
-          </geometry>
-          <material name="rubber">
-             <color rgba="0.1 0.1 0.1 1" />
-          </material>
+          <mass value="0.1" />
+          <inertia
+            ixx="0.0000729"
+            ixy="0"
+            ixz="0"
+            iyy="0.0000729"
+            iyz="0"
+            izz="0.0001458"
+          />
+        </inertial>
+        <visual>
+          <geometry>
+            <cylinder radius="0.054" length="0.043" />
+          </geometry>
+          <material name="rubber"/>
         </visual>
         <collision name='collision'>
@@ -115,12 +119,60 @@
       <link name="rear_right_wheel">
         <inertial>
-          <mass value="2.0" />
-          <inertia
-            ixx="0.145833"
-            ixy="0"
-            ixz="0"
-            iyy="0.145833"
-            iyz="0"
-            izz="0.125"
+          <mass value="0.1" />
+          <inertia
+            ixx="0.0000729"
+            ixy="0"
+            ixz="0"
+            iyy="0.0000729"
+            iyz="0"
+            izz="0.0001458"
+          />
+        </inertial>
+        <visual>
+          <geometry>
+            <cylinder radius="0.054" length="0.043" />
+          </geometry>
+          <material name="rubber"/>
+        </visual>
+        <collision name='collision'>
+          <geometry>
+            <cylinder radius="0.054" length="0.043" />
+          </geometry>
+        </collision>
+      </link>
+      <link name="front_left_wheel">
+        <inertial>
+          <mass value="0.1" />
+          <inertia
+            ixx="0.0000729"
+            ixy="0"
+            ixz="0"
+            iyy="0.0000729"
+            iyz="0"
+            izz="0.0001458"
+          />
+        </inertial>
+        <visual>
+          <geometry>
+            <cylinder radius="0.054" length="0.043" />
+          </geometry>
+          <material name="rubber"/>
+        </visual>
+        <collision name='collision'>
+          <geometry>
+            <cylinder radius="0.054" length="0.043" />
+          </geometry>
+        </collision>
+      </link>
+      <link name="front_right_wheel">
+        <inertial>
+          <mass value="0.1" />
+          <inertia
+            ixx="0.0000729"
+            ixy="0"
+            ixz="0"
+            iyy="0.0000729"
+            iyz="0"
+            izz="0.0001458"
           />
         </inertial>
@@ -137,64 +189,14 @@
         </collision>
       </link>
-      <link name="front_left_wheel">
-        <inertial>
-          <mass value="2.0" />
-          <inertia
-            ixx="0.145833"
-            ixy="0"
-            ixz="0"
-            iyy="0.145833"
-            iyz="0"
-            izz="0.125"
-          />
-        </inertial>
-        <visual>
-          <geometry>
-            <cylinder radius="0.054" length="0.043" />
-          </geometry>
-          <material name="rubber">
-             <color rgba="1.0 1.0 1.0 1.0" />
-          </material>
-        </visual>
-        <collision name='collision'>
-          <geometry>
-            <cylinder radius="0.054" length="0.043" />
-          </geometry>
-        </collision>
-      </link>
-      <link name="front_right_wheel">
-        <inertial>
-          <mass value="2.0" />
-          <inertia
-            ixx="0.145833"
-            ixy="0"
-            ixz="0"
-            iyy="0.145833"
-            iyz="0"
-            izz="0.125"
-          />
-        </inertial>
-        <visual>
-          <geometry>
-            <cylinder radius="0.054" length="0.043" />
-          </geometry>
-          <material name="rubber" />
-        </visual>
-        <collision name='collision'>
-          <geometry>
-            <cylinder radius="0.054" length="0.043" />
-          </geometry>
-        </collision>
-      </link>
       <link name="front_left_hub">
         <inertial>
-          <mass value="0.0001" />
-          <inertia
-            ixx="0.001"
-            ixy="0"
-            ixz="0"
-            iyy="0.001"
-            iyz="0"
-            izz="0.001"
+          <mass value="0.0" />
+          <inertia
+            ixx="0.0"
+            ixy="0"
+            ixz="0"
+            iyy="0.0"
+            iyz="0"
+            izz="0.0"
           />
         </inertial>
@@ -207,12 +209,12 @@
       <link name="front_right_hub">
         <inertial>
-          <mass value="0.0001" />
-          <inertia
-            ixx="0.001"
-            ixy="0"
-            ixz="0"
-            iyy="0.001"
-            iyz="0"
-            izz="0.001"
+          <mass value="0.0" />
+          <inertia
+            ixx="0.0"
+            ixy="0"
+            ixz="0"
+            iyy="0.0"
+            iyz="0"
+            izz="0.0"
           />
         </inertial>
@@ -271,4 +273,3 @@
         <axis xyz="0 0 1" />
       </joint>
-      <xacro:include filename="$(find rviz_description)/urdf/car.gazebo.xacro" />
 </robot>

Commit message: Added odometry, tire physics to simulation, created steering testing launch file

File: rviz_description/urdf/car.urdf.xacro (robot description, xacro)
@@ -261,5 +261,5 @@
       <joint name="front_left_hub_joint" type="revolute">
         <origin xyz="0.14 0.11 0.054" rpy="0 0 0" />
-        <limit effort="1000" upper="0.5" lower="-0.5" velocity="100.0" />
+        <limit upper="0.5" lower="-0.5" velocity="2.0" />
         <parent link="base_link" />
         <child link="front_left_hub" />
@@ -268,5 +268,5 @@
       <joint name="front_right_hub_joint" type="revolute">
         <origin xyz="0.14 -0.11 0.054" rpy="0 0 0" />
-        <limit effort="1000" upper="0.5" lower="-0.5" velocity="100.0" />
+        <limit upper="0.5" lower="-0.5" velocity="2.0" />
         <parent link="base_link" />
         <child link="front_right_hub" />
